Commit message: real time calibration with camera vid input

File: ABH_URDF/ability_hand.urdf (robot description, URDF)
Before this commit: robot ability_hand, 11 links, 10 joints
Links:
- link index_L1: geometry visual mesh filename=models/idx-F1.STL
- link index_L2: geometry visual mesh filename=models/idx-F2.STL
- link middle_L1: geometry visual mesh filename=models/idx-F1.STL
- link middle_L2: geometry visual mesh filename=models/idx-F2.STL
- link pinky_L1: geometry visual mesh filename=models/idx-F1.STL
- link pinky_L2: geometry visual mesh filename=models/idx-F2.STL
- link ring_L1: geometry visual mesh filename=models/idx-F1.STL
- link ring_L2: geometry visual mesh filename=models/idx-F2.STL
- link thumb_L1: geometry visual mesh filename=models/thumb-F1.STL
- link thumb_L2: geometry visual mesh filename=models/thumb-F2.STL
